File: dropbot-v3-connection-adapter.kicad_pcb (KiCad board)
At the start: 2 copper layers, 76 x 50.8 mm, 142 parts, among them J1 CONN_02X20, J2 CONN_02X25, J3 CONN_02X20, P1 CONN_01X01, P10 CONN_01X01, P100 CONN_01X01, P101 CONN_01X01, P102 CONN_01X01, P103 CONN_01X01, P104 CONN_01X01, P105 CONN_01X01, P106 CONN_01X01, P107 CONN_01X01, P108 CONN_01X01, P109 CONN_01X01, P11 CONN_01X01, P110 CONN_01X01, P111 CONN_01X01, P112 CONN_01X01, P113 CONN_01X01, P114 CONN_01X01, P115 CONN_01X01, P116 CONN_01X01, P117 CONN_01X01, P118 CONN_01X01, P119 CONN_01X01, P12 CONN_01X01, P120 CONN_01X01, P122 CONN_01X01, P123 CONN_01X01, P124 CONN_01X01, P125 CONN_01X01, P126 CONN_01X01, P127 CONN_01X01, P128 CONN_01X01, P129 CONN_01X01, P13 CONN_01X01, P130 CONN_01X01, P131 CONN_01X01, P132 CONN_01X01, P133 CONN_01X01, P134 CONN_01X01, P135 CONN_01X01, P136 CONN_01X01, P137 CONN_01X01, P14 CONN_01X01, P15 CONN_01X01, P16 CONN_01X01, P17 CONN_01X01, P18 CONN_01X01, P19 CONN_01X01, P2 CONN_01X01, P20 CONN_01X01, P21 CONN_01X01, P22 CONN_01X01, P23 CONN_01X01, P24 CONN_01X01, P25 CONN_01X01, P26 CONN_01X01, P27 CONN_01X01, P28 CONN_01X01, P29 CONN_01X01, P3 CONN_01X01, P30 CONN_01X01, P31 CONN_01X01, P32 CONN_01X01, P33 CONN_01X01, P34 CONN_01X01, P35 CONN_01X01, P36 CONN_01X01, P37 CONN_01X01, P38 CONN_01X01, P39 CONN_01X01, P4 CONN_01X01, P40 CONN_01X01, P41 CONN_01X01, P42 CONN_01X01, P43 CONN_01X01, P44 CONN_01X01, P45 CONN_01X01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

Commit message: Fix connector orientation
Parts:
- moved J2 1.23 mm to (76.3, 58.4), turned to 90 degrees
- turned J1 to 90 degrees
- turned J3 to 90 degrees
Connections:
- P1 pad 1: Net-(J1-Pad1) -> Net-(J1-Pad40)
- P10 pad 1: Net-(J1-Pad10) -> Net-(J1-Pad31)
- P100 pad 1: Net-(J3-Pad20) -> Net-(J3-Pad21)
- P101 pad 1: Net-(J3-Pad21) -> Net-(J3-Pad20)
- P102 pad 1: Net-(J3-Pad22) -> Net-(J3-Pad19)
- P103 pad 1: Net-(J3-Pad23) -> Net-(J3-Pad18)
- P104 pad 1: Net-(J3-Pad24) -> Net-(J3-Pad17)
- P105 pad 1: Net-(J3-Pad25) -> Net-(J3-Pad16)
- P106 pad 1: Net-(J3-Pad26) -> Net-(J3-Pad15)
- P107 pad 1: Net-(J3-Pad27) -> Net-(J3-Pad14)
- P108 pad 1: Net-(J3-Pad28) -> Net-(J3-Pad13)
- P109 pad 1: Net-(J3-Pad29) -> Net-(J3-Pad12)
- P11 pad 1: Net-(J1-Pad11) -> Net-(J1-Pad30)
- P110 pad 1: Net-(J3-Pad30) -> Net-(J3-Pad11)
- P111 pad 1: Net-(J3-Pad31) -> Net-(J3-Pad10)
- P112 pad 1: Net-(J3-Pad32) -> Net-(J3-Pad9)
- P113 pad 1: Net-(J3-Pad33) -> Net-(J3-Pad8)
- P114 pad 1: Net-(J3-Pad34) -> Net-(J3-Pad7)
- P115 pad 1: Net-(J3-Pad35) -> Net-(J3-Pad6)
- P116 pad 1: Net-(J3-Pad36) -> Net-(J3-Pad5)
- P117 pad 1: Net-(J3-Pad37) -> Net-(J3-Pad4)
- P118 pad 1: Net-(J3-Pad38) -> Net-(J3-Pad3)
- P119 pad 1: Net-(J3-Pad39) -> Net-(J3-Pad2)
- P12 pad 1: Net-(J1-Pad12) -> Net-(J1-Pad29)
- P120 pad 1: Net-(J3-Pad40) -> Net-(J3-Pad1)
- P122 pad 1: CUR_SENSE -> Net-(P122-Pad1)
- P123 pad 1: GND -> Net-(P123-Pad1)
- P124 pad 1: HV_OE -> Net-(P124-Pad1)
- P13 pad 1: Net-(J1-Pad13) -> Net-(J1-Pad28)
- P130 pad 1: Net-(P130-Pad1) -> CUR_SENSE
- P131 pad 1: Net-(P131-Pad1) -> GND
- P132 pad 1: Net-(P132-Pad1) -> HV_OE
- P14 pad 1: Net-(J1-Pad14) -> Net-(J1-Pad27)
- P15 pad 1: Net-(J1-Pad15) -> Net-(J1-Pad26)
- P16 pad 1: Net-(J1-Pad16) -> Net-(J1-Pad25)
- P17 pad 1: Net-(J1-Pad17) -> Net-(J1-Pad24)
- P18 pad 1: Net-(J1-Pad18) -> Net-(J1-Pad23)
- P19 pad 1: Net-(J1-Pad19) -> Net-(J1-Pad22)
- P2 pad 1: Net-(J1-Pad2) -> Net-(J1-Pad39)
- P20 pad 1: Net-(J1-Pad20) -> Net-(J1-Pad21)
- P21 pad 1: Net-(J1-Pad21) -> Net-(J1-Pad20)
- P22 pad 1: Net-(J1-Pad22) -> Net-(J1-Pad19)
- P23 pad 1: Net-(J1-Pad23) -> Net-(J1-Pad18)
- P24 pad 1: Net-(J1-Pad24) -> Net-(J1-Pad17)
- P25 pad 1: Net-(J1-Pad25) -> Net-(J1-Pad16)
- P26 pad 1: Net-(J1-Pad26) -> Net-(J1-Pad15)
- P27 pad 1: Net-(J1-Pad27) -> Net-(J1-Pad14)
- P28 pad 1: Net-(J1-Pad28) -> Net-(J1-Pad13)
- P29 pad 1: Net-(J1-Pad29) -> Net-(J1-Pad12)
- P3 pad 1: Net-(J1-Pad3) -> Net-(J1-Pad38)
- P30 pad 1: Net-(J1-Pad30) -> Net-(J1-Pad11)
- P31 pad 1: Net-(J1-Pad31) -> Net-(J1-Pad10)
- P32 pad 1: Net-(J1-Pad32) -> Net-(J1-Pad9)
- P33 pad 1: Net-(J1-Pad33) -> Net-(J1-Pad8)
- P34 pad 1: Net-(J1-Pad34) -> Net-(J1-Pad7)
- P35 pad 1: Net-(J1-Pad35) -> Net-(J1-Pad6)
- P36 pad 1: Net-(J1-Pad36) -> Net-(J1-Pad5)
- P37 pad 1: Net-(J1-Pad37) -> Net-(J1-Pad4)
- P38 pad 1: Net-(J1-Pad38) -> Net-(J1-Pad3)
- P39 pad 1: Net-(J1-Pad39) -> Net-(J1-Pad2)
- P4 pad 1: Net-(J1-Pad4) -> Net-(J1-Pad37)
- P40 pad 1: Net-(J1-Pad40) -> Net-(J1-Pad1)
- P41 pad 1: Net-(J2-Pad11) -> Net-(J2-Pad50)
- P42 pad 1: Net-(J2-Pad12) -> Net-(J2-Pad49)
- P43 pad 1: Net-(J2-Pad13) -> Net-(J2-Pad48)
- P44 pad 1: Net-(J2-Pad14) -> Net-(J2-Pad47)
- P45 pad 1: Net-(J2-Pad15) -> Net-(J2-Pad46)
- P46 pad 1: Net-(J2-Pad16) -> Net-(J2-Pad45)
- P47 pad 1: Net-(J2-Pad17) -> Net-(J2-Pad44)
- P48 pad 1: Net-(J2-Pad18) -> Net-(J2-Pad43)
- P49 pad 1: Net-(J2-Pad19) -> Net-(J2-Pad42)
- P5 pad 1: Net-(J1-Pad5) -> Net-(J1-Pad36)
- P50 pad 1: Net-(J2-Pad20) -> Net-(J2-Pad41)
- P51 pad 1: Net-(J2-Pad21) -> Net-(J2-Pad40)
- P52 pad 1: Net-(J2-Pad22) -> Net-(J2-Pad39)
- P53 pad 1: Net-(J2-Pad23) -> Net-(J2-Pad38)
- P54 pad 1: Net-(J2-Pad24) -> Net-(J2-Pad37)
- P55 pad 1: Net-(J2-Pad25) -> Net-(J2-Pad36)
- P56 pad 1: Net-(J2-Pad26) -> Net-(J2-Pad35)
- P57 pad 1: Net-(J2-Pad27) -> Net-(J2-Pad34)
- P58 pad 1: Net-(J2-Pad28) -> Net-(J2-Pad33)
- P59 pad 1: Net-(J2-Pad29) -> Net-(J2-Pad32)
- P6 pad 1: Net-(J1-Pad6) -> Net-(J1-Pad35)
- P60 pad 1: Net-(J2-Pad30) -> Net-(J2-Pad31)
- P61 pad 1: Net-(J2-Pad31) -> Net-(J2-Pad30)
- P62 pad 1: Net-(J2-Pad32) -> Net-(J2-Pad29)
- P63 pad 1: Net-(J2-Pad33) -> Net-(J2-Pad28)
- P64 pad 1: Net-(J2-Pad34) -> Net-(J2-Pad27)
- P65 pad 1: Net-(J2-Pad35) -> Net-(J2-Pad26)
- P66 pad 1: Net-(J2-Pad36) -> Net-(J2-Pad25)
- P67 pad 1: Net-(J2-Pad37) -> Net-(J2-Pad24)
- P68 pad 1: Net-(J2-Pad38) -> Net-(J2-Pad23)
- P69 pad 1: Net-(J2-Pad39) -> Net-(J2-Pad22)
- P7 pad 1: Net-(J1-Pad7) -> Net-(J1-Pad34)
- P70 pad 1: Net-(J2-Pad40) -> Net-(J2-Pad21)
- P71 pad 1: Net-(J2-Pad41) -> Net-(J2-Pad20)
- P72 pad 1: Net-(J2-Pad42) -> Net-(J2-Pad19)
- P73 pad 1: Net-(J2-Pad43) -> Net-(J2-Pad18)
- P74 pad 1: Net-(J2-Pad44) -> Net-(J2-Pad17)
- P75 pad 1: Net-(J2-Pad45) -> Net-(J2-Pad16)
- P76 pad 1: Net-(J2-Pad46) -> Net-(J2-Pad15)
- P77 pad 1: Net-(J2-Pad47) -> Net-(J2-Pad14)
- P78 pad 1: Net-(J2-Pad48) -> Net-(J2-Pad13)
- P79 pad 1: Net-(J2-Pad49) -> Net-(J2-Pad12)
- P8 pad 1: Net-(J1-Pad8) -> Net-(J1-Pad33)
- P80 pad 1: Net-(J2-Pad50) -> Net-(J2-Pad11)
- P81 pad 1: Net-(J3-Pad1) -> Net-(J3-Pad40)
- P82 pad 1: Net-(J3-Pad2) -> Net-(J3-Pad39)
- P83 pad 1: Net-(J3-Pad3) -> Net-(J3-Pad38)
- P84 pad 1: Net-(J3-Pad4) -> Net-(J3-Pad37)
- P85 pad 1: Net-(J3-Pad5) -> Net-(J3-Pad36)
- P86 pad 1: Net-(J3-Pad6) -> Net-(J3-Pad35)
- P87 pad 1: Net-(J3-Pad7) -> Net-(J3-Pad34)
- P88 pad 1: Net-(J3-Pad8) -> Net-(J3-Pad33)
- P89 pad 1: Net-(J3-Pad9) -> Net-(J3-Pad32)
- P9 pad 1: Net-(J1-Pad9) -> Net-(J1-Pad32)
- P90 pad 1: Net-(J3-Pad10) -> Net-(J3-Pad31)
- P91 pad 1: Net-(J3-Pad11) -> Net-(J3-Pad30)
- P92 pad 1: Net-(J3-Pad12) -> Net-(J3-Pad29)
- P93 pad 1: Net-(J3-Pad13) -> Net-(J3-Pad28)
- P94 pad 1: Net-(J3-Pad14) -> Net-(J3-Pad27)
- P95 pad 1: Net-(J3-Pad15) -> Net-(J3-Pad26)
- P96 pad 1: Net-(J3-Pad16) -> Net-(J3-Pad25)
- P97 pad 1: Net-(J3-Pad17) -> Net-(J3-Pad24)
- P98 pad 1: Net-(J3-Pad18) -> Net-(J3-Pad23)
- P99 pad 1: Net-(J3-Pad19) -> Net-(J3-Pad22)
Routing:
- net GND: track 3.91 -> 101.3 mm, vias 2 -> 6
- net Net-(J3-Pad25): track 63.8 -> 21.6 mm
- net Net-(J3-Pad16): track 21.6 -> 62.3 mm
- net Net-(J3-Pad26): track 50.3 -> 16.1 mm
- net Net-(J3-Pad37): track 70.7 -> 36.6 mm, vias 2 -> 4
- net Net-(J3-Pad4): track 36.6 -> 70.7 mm, vias 4 -> 2
- net Net-(J3-Pad15): track 16.1 -> 50.1 mm
- net Net-(J3-Pad33): track 66.3 -> 33.5 mm, vias 2 -> 4
- net Net-(J3-Pad8): track 33.5 -> 66.3 mm, vias 4 -> 2
- net Net-(J3-Pad29): track 62.3 -> 30.3 mm, vias 2 -> 4
- net Net-(J3-Pad12): track 30.3 -> 62.3 mm, vias 4 -> 2
- net Net-(J2-Pad50): track 34.7 -> 66.7 mm
- net Net-(J3-Pad3): track 31.7 -> 61.2 mm
- net Net-(J3-Pad38): track 61.2 -> 31.7 mm
- net Net-(J2-Pad49): track 33.7 -> 62.7 mm
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Other:
- board text added: "DropBot v3 connection adapter v1.1 http://sci-bots.com 2019"
- board text removed: "DropBot v3 connection adapter v1.0 http://sci-bots.com 2019"
