File: dropbot-v3-connection-adapter.sch (KiCad schematic (older format))
At the start: 139 parts, among them J1 CONN_02X20, J2 CONN_02X25, J3 CONN_02X20, P1 CONN_01X01, P10 CONN_01X01, P100 CONN_01X01, P101 CONN_01X01, P102 CONN_01X01, P103 CONN_01X01, P104 CONN_01X01, P105 CONN_01X01, P106 CONN_01X01, P107 CONN_01X01, P108 CONN_01X01, P109 CONN_01X01, P11 CONN_01X01, P110 CONN_01X01, P111 CONN_01X01, P112 CONN_01X01, P113 CONN_01X01, P114 CONN_01X01, P115 CONN_01X01, P116 CONN_01X01, P117 CONN_01X01, P118 CONN_01X01, P119 CONN_01X01, P12 CONN_01X01, P120 CONN_01X01, P122 CONN_01X01, P123 CONN_01X01, P124 CONN_01X01, P125 CONN_01X01, P126 CONN_01X01, P127 CONN_01X01, P128 CONN_01X01, P129 CONN_01X01, P13 CONN_01X01, P130 CONN_01X01, P131 CONN_01X01, P132 CONN_01X01, P133 CONN_01X01, P134 CONN_01X01, P135 CONN_01X01, P136 CONN_01X01, P137 CONN_01X01, P14 CONN_01X01, P15 CONN_01X01, P16 CONN_01X01, P17 CONN_01X01, P18 CONN_01X01, P19 CONN_01X01, P2 CONN_01X01, P20 CONN_01X01, P21 CONN_01X01, P22 CONN_01X01, P23 CONN_01X01, P24 CONN_01X01, P25 CONN_01X01, P26 CONN_01X01, P27 CONN_01X01, P28 CONN_01X01, P29 CONN_01X01, P3 CONN_01X01, P30 CONN_01X01, P31 CONN_01X01, P32 CONN_01X01, P33 CONN_01X01, P34 CONN_01X01, P35 CONN_01X01, P36 CONN_01X01, P37 CONN_01X01, P38 CONN_01X01, P39 CONN_01X01, P4 CONN_01X01, P40 CONN_01X01, P41 CONN_01X01, P42 CONN_01X01, P43 CONN_01X01, P44 CONN_01X01, P45 CONN_01X01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

Commit message: Fix connector orientation
Parts:
- J1, J3: symbol CONN_02X20 -> dropbot-v3-connection-adapter-rescue:CONN_02X20
- J2: symbol CONN_02X25 -> dropbot-v3-connection-adapter-rescue:CONN_02X25
- P1, P10, P100, P101, P102, P103, P104, P105, P106, P107, P108, P109, P11, P110, P111, P112, P113, P114, P115, P116, P117, P118, P119, P12, P120, P122, P123, P124, P125, P126, P127, P128, P129, P13, P130, P131, P132, P133, P134, P135, P136, P137, P14, P15, P16, P17, P18, P19, P2, P20, P21, P22, P23, P24, P25, P26, P27, P28, P29, P3, P30, P31, P32, P33, P34, P35, P36, P37, P38, P39, P4, P40, P41, P42, P43, P44, P45, P46, P47, P48, P49, P5, P50, P51, P52, P53, P54, P55, P56, P57, P58, P59, P6, P60, P61, P62, P63, P64, P65, P66, P67, P68, P69, P7, P70, P71, P72, P73, P74, P75, P76, P77, P78, P79, P8, P80, P81, P82, P83, P84, P85, P86, P87, P88, P89, P9, P90, P91, P92, P93, P94, P95, P96, P97, P98, P99: symbol CONN_01X01 -> dropbot-v3-connection-adapter-rescue:CONN_01X01
Connections:
- net CUR_SENSE: now also P130.1 (P1); no longer P122.1 (P1)
- net GND: now also P131.1 (P1); no longer P123.1 (P1)
- net HV_OE: now also P132.1 (P1); no longer P124.1 (P1)
- net at P1.1 (P1): now also J1.40 (P40); no longer J1.1 (P1)
- net at P2.1 (P1): now also J1.39 (P39); no longer J1.2 (P2)
- net at P3.1 (P1): now also J1.38 (P38); no longer J1.3 (P3)
- net at P4.1 (P1): now also J1.37 (P37); no longer J1.4 (P4)
- net at P5.1 (P1): now also J1.36 (P36); no longer J1.5 (P5)
- net at P6.1 (P1): now also J1.35 (P35); no longer J1.6 (P6)
- net at P7.1 (P1): now also J1.34 (P34); no longer J1.7 (P7)
- net at P8.1 (P1): now also J1.33 (P33); no longer J1.8 (P8)
- net at P9.1 (P1): now also J1.32 (P32); no longer J1.9 (P9)
- net at P10.1 (P1): now also J1.31 (P31); no longer J1.10 (P10)
- net at P11.1 (P1): now also J1.30 (P30); no longer J1.11 (P11)
- net at P12.1 (P1): now also J1.29 (P29); no longer J1.12 (P12)
- net at P13.1 (P1): now also J1.28 (P28); no longer J1.13 (P13)
- net at P14.1 (P1): now also J1.27 (P27); no longer J1.14 (P14)
- net at P15.1 (P1): now also J1.26 (P26); no longer J1.15 (P15)
- net at P16.1 (P1): now also J1.25 (P25); no longer J1.16 (P16)
- net at P17.1 (P1): now also J1.24 (P24); no longer J1.17 (P17)
- net at P18.1 (P1): now also J1.23 (P23); no longer J1.18 (P18)
- net at P19.1 (P1): now also J1.22 (P22); no longer J1.19 (P19)
- net at P20.1 (P1): now also J1.21 (P21); no longer J1.20 (P20)
- net at P21.1 (P1): now also J1.20 (P20); no longer J1.21 (P21)
- net at P22.1 (P1): now also J1.19 (P19); no longer J1.22 (P22)
- net at P23.1 (P1): now also J1.18 (P18); no longer J1.23 (P23)
- net at P24.1 (P1): now also J1.17 (P17); no longer J1.24 (P24)
- net at P25.1 (P1): now also J1.16 (P16); no longer J1.25 (P25)
- net at P26.1 (P1): now also J1.15 (P15); no longer J1.26 (P26)
- net at P27.1 (P1): now also J1.14 (P14); no longer J1.27 (P27)
- net at P28.1 (P1): now also J1.13 (P13); no longer J1.28 (P28)
- net at P29.1 (P1): now also J1.12 (P12); no longer J1.29 (P29)
- net at P30.1 (P1): now also J1.11 (P11); no longer J1.30 (P30)
- net at P31.1 (P1): now also J1.10 (P10); no longer J1.31 (P31)
- net at P32.1 (P1): now also J1.9 (P9); no longer J1.32 (P32)
- net at P33.1 (P1): now also J1.8 (P8); no longer J1.33 (P33)
- net at P34.1 (P1): now also J1.7 (P7); no longer J1.34 (P34)
- net at P35.1 (P1): now also J1.6 (P6); no longer J1.35 (P35)
- net at P36.1 (P1): now also J1.5 (P5); no longer J1.36 (P36)
- net at P37.1 (P1): now also J1.4 (P4); no longer J1.37 (P37)
- net at P38.1 (P1): now also J1.3 (P3); no longer J1.38 (P38)
- net at P39.1 (P1): now also J1.2 (P2); no longer J1.39 (P39)
- net at P40.1 (P1): now also J1.1 (P1); no longer J1.40 (P40)
- net at P41.1 (P1): now also J2.50 (P50); no longer J2.11 (P11)
- net at P42.1 (P1): now also J2.49 (P49); no longer J2.12 (P12)
- net at P43.1 (P1): now also J2.48 (P48); no longer J2.13 (P13)
- net at P44.1 (P1): now also J2.47 (P47); no longer J2.14 (P14)
- net at P45.1 (P1): now also J2.46 (P46); no longer J2.15 (P15)
- net at P46.1 (P1): now also J2.45 (P45); no longer J2.16 (P16)
- net at P47.1 (P1): now also J2.44 (P44); no longer J2.17 (P17)
- net at P48.1 (P1): now also J2.43 (P43); no longer J2.18 (P18)
- net at P49.1 (P1): now also J2.42 (P42); no longer J2.19 (P19)
- net at P50.1 (P1): now also J2.41 (P41); no longer J2.20 (P20)
- net at P51.1 (P1): now also J2.40 (P40); no longer J2.21 (P21)
- net at P52.1 (P1): now also J2.39 (P39); no longer J2.22 (P22)
- net at P53.1 (P1): now also J2.38 (P38); no longer J2.23 (P23)
- net at P54.1 (P1): now also J2.37 (P37); no longer J2.24 (P24)
- net at P55.1 (P1): now also J2.36 (P36); no longer J2.25 (P25)
- net at P56.1 (P1): now also J2.35 (P35); no longer J2.26 (P26)
- net at P57.1 (P1): now also J2.34 (P34); no longer J2.27 (P27)
- net at P58.1 (P1): now also J2.33 (P33); no longer J2.28 (P28)
- net at P59.1 (P1): now also J2.32 (P32); no longer J2.29 (P29)
- net at P60.1 (P1): now also J2.31 (P31); no longer J2.30 (P30)
- net at P61.1 (P1): now also J2.30 (P30); no longer J2.31 (P31)
- net at P62.1 (P1): now also J2.29 (P29); no longer J2.32 (P32)
- net at P63.1 (P1): now also J2.28 (P28); no longer J2.33 (P33)
- net at P64.1 (P1): now also J2.27 (P27); no longer J2.34 (P34)
- net at P65.1 (P1): now also J2.26 (P26); no longer J2.35 (P35)
- net at P66.1 (P1): now also J2.25 (P25); no longer J2.36 (P36)
- net at P67.1 (P1): now also J2.24 (P24); no longer J2.37 (P37)
- net at P68.1 (P1): now also J2.23 (P23); no longer J2.38 (P38)
- net at P69.1 (P1): now also J2.22 (P22); no longer J2.39 (P39)
- net at P70.1 (P1): now also J2.21 (P21); no longer J2.40 (P40)
- net at P71.1 (P1): now also J2.20 (P20); no longer J2.41 (P41)
- net at P72.1 (P1): now also J2.19 (P19); no longer J2.42 (P42)
- net at P73.1 (P1): now also J2.18 (P18); no longer J2.43 (P43)
- net at P74.1 (P1): now also J2.17 (P17); no longer J2.44 (P44)
- net at P75.1 (P1): now also J2.16 (P16); no longer J2.45 (P45)
- net at P76.1 (P1): now also J2.15 (P15); no longer J2.46 (P46)
- net at P77.1 (P1): now also J2.14 (P14); no longer J2.47 (P47)
- net at P78.1 (P1): now also J2.13 (P13); no longer J2.48 (P48)
- net at P79.1 (P1): now also J2.12 (P12); no longer J2.49 (P49)
- net at P80.1 (P1): now also J2.11 (P11); no longer J2.50 (P50)
- net at P81.1 (P1): now also J3.40 (P40); no longer J3.1 (P1)
- net at P82.1 (P1): now also J3.39 (P39); no longer J3.2 (P2)
- net at P83.1 (P1): now also J3.38 (P38); no longer J3.3 (P3)
- net at P84.1 (P1): now also J3.37 (P37); no longer J3.4 (P4)
- net at P85.1 (P1): now also J3.36 (P36); no longer J3.5 (P5)
- net at P86.1 (P1): now also J3.35 (P35); no longer J3.6 (P6)
- net at P87.1 (P1): now also J3.34 (P34); no longer J3.7 (P7)
- net at P88.1 (P1): now also J3.33 (P33); no longer J3.8 (P8)
- net at P89.1 (P1): now also J3.32 (P32); no longer J3.9 (P9)
- net at P90.1 (P1): now also J3.31 (P31); no longer J3.10 (P10)
- net at P91.1 (P1): now also J3.30 (P30); no longer J3.11 (P11)
- net at P92.1 (P1): now also J3.29 (P29); no longer J3.12 (P12)
- net at P93.1 (P1): now also J3.28 (P28); no longer J3.13 (P13)
- net at P94.1 (P1): now also J3.27 (P27); no longer J3.14 (P14)
- net at P95.1 (P1): now also J3.26 (P26); no longer J3.15 (P15)
- net at P96.1 (P1): now also J3.25 (P25); no longer J3.16 (P16)
- net at P97.1 (P1): now also J3.24 (P24); no longer J3.17 (P17)
- net at P98.1 (P1): now also J3.23 (P23); no longer J3.18 (P18)
- net at P99.1 (P1): now also J3.22 (P22); no longer J3.19 (P19)
- net at P100.1 (P1): now also J3.21 (P21); no longer J3.20 (P20)
- net at P101.1 (P1): now also J3.20 (P20); no longer J3.21 (P21)
- net at P102.1 (P1): now also J3.19 (P19); no longer J3.22 (P22)
- net at P103.1 (P1): now also J3.18 (P18); no longer J3.23 (P23)
- net at P104.1 (P1): now also J3.17 (P17); no longer J3.24 (P24)
- net at P105.1 (P1): now also J3.16 (P16); no longer J3.25 (P25)
- net at P106.1 (P1): now also J3.15 (P15); no longer J3.26 (P26)
- net at P107.1 (P1): now also J3.14 (P14); no longer J3.27 (P27)
- net at P108.1 (P1): now also J3.13 (P13); no longer J3.28 (P28)
- net at P109.1 (P1): now also J3.12 (P12); no longer J3.29 (P29)
- net at P110.1 (P1): now also J3.11 (P11); no longer J3.30 (P30)
- net at P111.1 (P1): now also J3.10 (P10); no longer J3.31 (P31)
- net at P112.1 (P1): now also J3.9 (P9); no longer J3.32 (P32)
- net at P113.1 (P1): now also J3.8 (P8); no longer J3.33 (P33)
- net at P114.1 (P1): now also J3.7 (P7); no longer J3.34 (P34)
- net at P115.1 (P1): now also J3.6 (P6); no longer J3.35 (P35)
- net at P116.1 (P1): now also J3.5 (P5); no longer J3.36 (P36)
- net at P117.1 (P1): now also J3.4 (P4); no longer J3.37 (P37)
- net at P118.1 (P1): now also J3.3 (P3); no longer J3.38 (P38)
- net at P119.1 (P1): now also J3.2 (P2); no longer J3.39 (P39)
- net at P120.1 (P1): now also J3.1 (P1); no longer J3.40 (P40)
Other:
- moved on the sheet: J2
